File: Case/southpawcase.kicad_pcb (KiCad board)
At the start: 2 copper layers, 376.2 x 109.5 mm, 4 parts

Commit message: Add feet mounting holes to the bottom plate
Parts:
- added REF**: MountingHole_4.3mm_M4_Pad, MountingHole:MountingHole_4.3mm_M4_Pad, F.Cu at (349.1, 115.2)
- added REF**: MountingHole_4.3mm_M4_Pad, MountingHole:MountingHole_4.3mm_M4_Pad, F.Cu at (72.9, 115.2)
- moved G*** 93.5 mm to (211.1, 145.4) (x2)
- moved G*** 93.5 mm to (47.6, 196.3) (x2)
Other:
- outline, holes or cut-outs redrawn
