File: ANSI+ISO_Plate/southpaw75-ansi-iso-plate.kicad_pcb (KiCad board)
At the start: 2 copper layers, 376.2 x 109.5 mm, 4 parts

Commit message: ANSI+ISO Plate: Update plate with rounded cutouts, split backspace and Tsangan support
Other:
- outline, holes or cut-outs redrawn
- net class Default removed
- board text added: "ANSI+ISO Plate RevF Modifications by piit79 / 42keebs.eu 2023"
- board text added: "Southpaw75"
